File: hardware/Alimentation.kicad_sch (KiCad schematic)
At the start: 6 parts, among them U3 AZ1117-3.3

Commit message: Encore plein de truc chouette
Other:
- company: Lang & Hiltpold SNC -> Lang & Hiltpold Software SNC
Changed lines of the file:
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@@
 		(title "STM32-DevBoard")
 		(date "2026-06-03")
-		(company "Lang & Hiltpold SNC")
+		(company "Lang & Hiltpold Software SNC")
 	)
 	(junction
