File: hardware/Rotary_Encorder.kicad_sch (KiCad schematic)
At the start: 10 parts, among them U4 AP2112R5-3.3TRG1

Commit message: Schema termine ?
Parts:
- removed C7: 10uF, symbol Device:C
- removed C8: 1uF, symbol Device:C
- removed D4, D5: LED, symbol Device:LED
- removed R28: 560, symbol Device:R
- removed R29: 220, symbol Device:R
- removed TP11: VBUS, symbol Connector:TestPoint
- removed TP12: 3v3, symbol Connector:TestPoint
- removed TP13: GND, symbol Connector:TestPoint
- removed U4: AP2112R5-3.3TRG1, RS_485_FOOT:AP2112R5-3.3, symbol RS_485_LIB:AP2112R5-3.3TRG1
- added C15, C16, C17: 10nF, symbol Device:C
- added R22, R23, R24, R25, R26, R27: 10k, symbol Device:R
- added S1: PEC12R-4217F-S0012, RS_485_FOOT:XDCR_PEC12R-4217F-S0012, symbol RS_485_LIB:PEC12R-4217F-S0012
Connections:
- net +3.3V: now also R22.1, R24.1, R26.1
- net GND: now also C15.2, C16.2, C17.2, S1.1, S1.C (COMMON), S1.SH1 (SHIELD), S1.SH2 (SHIELD__1)
- new net CHA: C15.1, R22.2, R23.1, S1.A (CHANNEL_A)
- new net CHB: C16.1, R24.2, R25.1, S1.B (CHANNEL_B)
- new net SW: C17.1, R26.2, R27.1, S1.2
- new net Switch: R27.2
- new net Terminal_A: R23.2
- new net Terminal_B: R25.2
- no-connect marks 1 -> 0

Commit message: Assignation terminee
Parts:
- C15, C16, C17: footprint (none) -> Capacitor_SMD:C_0805_2012Metric
- R22, R23, R24, R25, R26, R27: footprint (none) -> Resistor_SMD:R_0805_2012Metric
Changed lines of the file:
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@@
 			)
 		)
-		(property "Footprint" ""
+		(property "Footprint" "Resistor_SMD:R_0805_2012Metric"
 			(at 172.212 57.15 90)
 			(hide yes)
@@
 			)
 		)
-		(property "Footprint" ""
+		(property "Footprint" "Capacitor_SMD:C_0805_2012Metric"
 			(at 174.9552 121.92 0)
 			(hide yes)
@@
 			)
 		)
-		(property "Footprint" ""
+		(property "Footprint" "Resistor_SMD:R_0805_2012Metric"
 			(at 216.662 57.15 90)
 			(hide yes)
@@
 			)
 		)
-		(property "Footprint" ""
+		(property "Footprint" "Capacitor_SMD:C_0805_2012Metric"
 			(at 219.4052 76.2 0)
 			(hide yes)
@@
 			)
 		)
-		(property "Footprint" ""
+		(property "Footprint" "Resistor_SMD:R_0805_2012Metric"
 			(at 180.34 113.538 90)
 			(hide yes)
@@
 			)
 		)
-		(property "Footprint" ""
+		(property "Footprint" "Resistor_SMD:R_0805_2012Metric"
 			(at 180.34 67.818 90)
 			(hide yes)
@@
 			)
 		)
-		(property "Footprint" ""
+		(property "Footprint" "Resistor_SMD:R_0805_2012Metric"
 			(at 172.212 102.87 90)
 			(hide yes)
@@
 			)
 		)
-		(property "Footprint" ""
+		(property "Footprint" "Capacitor_SMD:C_0805_2012Metric"
 			(at 174.9552 76.2 0)
 			(hide yes)
@@
 			)
 		)
-		(property "Footprint" ""
+		(property "Footprint" "Resistor_SMD:R_0805_2012Metric"
 			(at 224.79 67.818 90)
 			(hide yes)
