File: hardware/STM32_DevBoard.kicad_sch (KiCad schematic)
At the start: 39 parts, among them SW1 SW_SPST, SW2 SW_MEC_5G, U1 STM32C071CBTx, U2 TP8485E-SR, U3 AZ1117-3.3, U4 HDC1080, U5 SGP40-D-R4

Commit message: encore plein de truc chouette
Parts:
- removed C1, C4: 100nF, symbol Device:C
- removed C5: 10uF, symbol Device:C
- removed C6: 22uF, symbol Device:C
- removed C8, C9: 1uF, symbol Device:C
- removed R1: 1M, symbol Device:R
- removed R6: 120, symbol Device:R
- removed R7: 0, symbol Device:R
- removed R8: 4.7, symbol Device:R
- removed TP10, TP11, TP12, TP13: GND, symbol Connector:TestPoint
- removed TP2: 3v3, symbol Connector:TestPoint
- removed TP3: VBUS, symbol Connector:TestPoint
- removed TP5: RS_458_B, symbol Connector:TestPoint
- removed TP6: RS_458_A, symbol Connector:TestPoint
- removed TP7: USART1_DE, symbol Connector:TestPoint
- removed TP8: USART1_RX, symbol Connector:TestPoint
- removed TP9: USART1_TX, symbol Connector:TestPoint
- removed U2: TP8485E-SR, RS_485_FOOT:SO-8SOIC-8_TPK, symbol RS_485_LIB:TP8485E-SR
- removed U3: AZ1117-3.3, Package_TO_SOT_SMD:SOT-223-3_TabPin2, symbol Regulator_Linear:AZ1117-3.3
- removed U4: HDC1080, Package_SON:Texas_PWSON-N6, symbol Sensor_Humidity:HDC1080
- removed U5: SGP40-D-R4, RS_485_FOOT:XCDR_SGP40-D-R4, symbol RS_485_LIB:SGP40-D-R4
- added C12: 100nF, symbol Device:C
- added LED1: IN-S66TBTRGB, RS_485_FOOT:IN-S66TB_INL, symbol RS_485_LIB:IN-S66TBTRGB
- added R13: 0, symbol Device:R
- added R14, R16: 360, symbol Device:R
- added R15: 560, symbol Device:R
- added TP15: GND, symbol Connector:TestPoint
- added TP16: SCL, symbol Connector:TestPoint
- added TP17: SDA, symbol Connector:TestPoint
- added TP18: VREF+, symbol Connector:TestPoint
- added U7: (no value), RS_485_FOOT:TFT_SPI, symbol RS_485_LIB:TFT_SPI
Connections:
- net +3.3V: now also R13.1, U7.1 (Vin)
- net GND: now also C12.2, TP15.1, U7.3 (GND)
- net I2C1_SCL: now also TP16.1
- net I2C1_SDA: now also TP17.1
- net VBUS: now also LED1.1
- net CC1_ADC: now reaches U1.13 (PA2)
- net CC2_ADC: now reaches U1.14 (PA3)
- net TIM14_CH1: now reaches U1.15 (PA4)
- net TIM14_CH1: now also U7.11 (Lite)
- net SPI1_SCK: now reaches U1.16 (PA5)
- net SPI1_SCK: now also U7.4 (SCK)
- net SPI1_MISO: now reaches U1.17 (PA6)
- net SPI1_MISO: now also U7.5 (MISO)
- net SPI1_MOSI: now reaches U1.18 (PA7)
- net SPI1_MOSI: now also U7.6 (MOSI)
- net PD0: now reaches U1.38 (PD0)
- net PD0: now also U7.7 (TFT_CS)
- net PD1: now reaches U1.39 (PD1)
- net PD1: now also U7.10 (SDCS)
- net PF3: now reaches U1.4 (PF3)
- net PF3: now also R14.2
- net PD2: now reaches U1.40 (PD2)
- net PD2: now also U7.9 (D/C)
- net PD3: now reaches U1.41 (PD3)
- net PD3: now also U7.8 (RST)
- net VREF+: now reaches U1.5 (VREF+)
- net VREF+: now also C12.1, R13.2, TP18.1
- net PF0: now reaches U1.8 (PF0)
- net PF0: now also R15.2
- net PF1: now reaches U1.9 (PF1)
- net PF1: now also R16.2
- new net: LED1.3, R14.1
- new net: LED1.2, R15.1
- new net: LED1.4, R16.1
- no-connect marks 37 -> 26
Other:
- added sheet Alimentation (Alimentation.kicad_sch)
- added sheet RS_485 (RS_485.kicad_sch)
- added sheet Sensors (Sensros.kicad_sch)
- sheet USB_Connector ports: added CC1_ADC, CC2_ADC; removed none
- moved on the sheet: C2, C3, C7, D1, R10, R4, R5, R9, SW1, SW2, TP1, TP14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

Commit message: Encore plein de truc chouette
Connections:
- net SWDIO: now reaches U1.35 (PA13)
- no-connect marks 26 -> 25
Other:
- company: Lang & Hiltpold SNC -> Lang & Hiltpold Software SNC
Changed lines of the file:
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@@
 		(title "STM32-DevBoard")
 		(date "2026-06-03")
-		(company "Lang & Hiltpold SNC")
+		(company "Lang & Hiltpold Software SNC")
 	)
 	(junction
@@
 	)
 	(no_connect
-		(at 173.99 85.09)
-	)
-	(no_connect
 		(at 173.99 128.27)
 	)
@@
 		(pts
 			(xy 54.61 46.99) (xy 54.61 40.64)
+		)
+		(stroke
+			(width 0)
+			(type default)
+		)
+	)
+	(wire
+		(pts
+			(xy 173.99 85.09) (xy 180.34 85.09)
 		)
 		(stroke
@@
 		(effects
 			(font
+				(size 1.27 1.27)
+			)
+			(justify left bottom)
+		)
+	)
+	(label "SWDIO"
+		(at 180.34 85.09 0)
+		(effects
+			(font

Commit message: Schema termine ?
Parts:
- added J4: (no value), Connector_PinHeader_1.27mm:PinHeader_2x07_P1.27mm_Horizontal, symbol RS_485_LIB:SWD_Interface
- added J5: Port_B_1, symbol Connector:Conn_01x08_Pin
- added J6: Port_B_2, symbol Connector:Conn_01x08_Pin
- renumbered C12 to C1, C7 to C2, C2 to C3, C3 to C4, R5 to R1, R9 to R2, R10 to R3, R13 to R5, R15 to R6, R16 to R7, R14 to R8, TP15 to TP1, TP17 to TP2, TP16 to TP3, TP1 to TP4, TP18 to TP5, TP4 to TP6, TP14 to TP7, U7 to U2
Connections:
- net +3.3V: now also J4.1 (3v3)
- net GND: now also J4.4 (GND)
- net SWDIO: now also J4.2 (SWDIO)
- net PC13: now reaches U1.1 (PC13)
- net at U1.19 (PB0): now also J5.8 (Pin_8)
- net at U1.20 (PB1): now also J5.7 (Pin_7)
- net at U1.21 (PB2): now also J5.6 (Pin_6)
- net at U1.22 (PB10): now also J6.6 (Pin_6)
- net at U1.23 (PB11): now also J6.5 (Pin_5)
- net at U1.24 (PB12): now also J6.4 (Pin_4)
- net at U1.25 (PB13): now also J6.3 (Pin_3)
- net at U1.26 (PB14): now also J6.2 (Pin_2)
- net at U1.27 (PB15): now also J6.1 (Pin_1)
- net PC6: now reaches U1.30 (PC6)
- net PC7: now reaches U1.31 (PC7)
- net at U1.42 (PB3): now also J5.5 (Pin_5)
- net at U1.43 (PB4): now also J5.4 (Pin_4)
- net at U1.44 (PB5): now also J5.3 (Pin_3)
- net at U1.45 (PB6): now also J5.2 (Pin_2)
- net at U1.46 (PB7): now also J5.1 (Pin_1)
- net at U1.47 (PB8): now also J6.8 (Pin_8)
- net at U1.48 (PB9): now also J6.7 (Pin_7)
- net BOOT0 renamed BOOT0 / SWCLK
- net BOOT0 / SWCLK: now also J4.3 (SWDCLK)
- no-connect marks 25 -> 6
Other:
- added sheet Rotary_Encorder (Rotary_Encorder.kicad_sch)
- sheet RS_485 ports: added none; removed +3.3V, GND
- sheet Sensors ports: added none; removed +3.3V, GND
- moved on the sheet: D1, R1, R4, SW1, TP4

Commit message: Assignation terminee
Parts:
- C1, C3, C4: footprint (none) -> Capacitor_SMD:C_0805_2012Metric
- C2: value 0.1uF -> 100nF; footprint (none) -> Capacitor_SMD:C_0805_2012Metric
- D1: value LED -> BOOT0_LED; footprint (none) -> LED_SMD:LED_0805_2012Metric
- J4: now left out of the parts list
- J5, J6: footprint (none) -> Connector_PinHeader_2.54mm:PinHeader_1x08_P2.54mm_Vertical
- R1, R2, R3, R4, R5, R6, R7, R8: footprint (none) -> Resistor_SMD:R_0805_2012Metric
- SW1: footprint (none) -> Button_Switch_THT:SW_PUSH_6mm
- SW2: footprint (none) -> Button_Switch_THT:SW_DIP_SPSTx01_Slide_6.7x4.1mm_W7.62mm_P2.54mm_LowProfile
- TP1, TP2, TP3, TP4, TP5, TP6, TP7: footprint (none) -> TestPoint:TestPoint_Loop_D2.50mm_Drill1.0mm
- U2: value (none) -> DISPLAY TFT
Other:
- sheet USB_Connector ports: added none; removed GND, VBUS
- moved on the sheet: D1, R1, TP4

Commit message: Start routing pcb
Parts:
- removed SW2: SW_MEC_5G, Button_Switch_THT:SW_DIP_SPSTx01_Slide_6.7x4.1mm_W7.62mm_P2.54mm_LowProfile, symbol Switch:SW_MEC_5G
- added SW2: SW_RESET, Button_Switch_THT:SW_PUSH_6mm, symbol Switch:SW_Push
- J4: footprint Connector_PinHeader_1.27mm:PinHeader_2x07_P1.27mm_Horizontal -> Connector_PinHeader_2.54mm:PinHeader_2x02_P2.54mm_Vertical
- SW1: value SW_SPST -> SW_BOOT; footprint Button_Switch_THT:SW_PUSH_6mm -> Button_Switch_THT:SW_DIP_SPSTx01_Slide_9.78x4.72mm_W7.62mm_P2.54mm
Connections:
- net GND: now also SW2.1
- net NRST: now also SW2.2
