File: hardware/STM32_DevBoard.kicad_pcb (KiCad board)
At the start: 4 copper layers, 134.6 x 42 mm, 101 parts, among them J1 USB4105-GF-A, J2 Screw_Terminal_01x02, J3 RJ45_LED_Shielded, J5 Port_B_1, J6 Port_B_2, SW1 SW_BOOT, SW2 SW_RESET, U1 STM32C071CBTx, U2 DISPLAY TFT, U3 USBLC6-2SC6, U4 AP2112R5-3.3TRG1, U5 SGP40-D-R4, U6 MS5607-02BA, U7 HDC1080, U8 TP8485E-SR

Commit message: PCB routing....
Parts:
- moved R18 211.8 mm to (218.5, 115.9), turned to 90 degrees
- moved R20 211.2 mm to (216.9, 121.5), turned to 180 degrees
- moved R21 210.2 mm to (216.9, 123.5), turned to 180 degrees
- moved R6 206.6 mm to (165.0, 112.2)
- moved TP15 206.0 mm to (199.0, 118.0)
- moved R7 205.6 mm to (165.0, 114.2)
- moved TP16 205.3 mm to (198.8, 122.0)
- moved R8 204.1 mm to (161.1, 116.2)
- moved TP17 201.1 mm to (199.0, 114.0)
- moved C13 199.2 mm to (222.0, 116.0), turned to 90 degrees
- moved R5 197.7 mm to (153.2, 101.7), turned to 90 degrees
- moved LED1 192.7 mm to (161.0, 113.8)
- moved TP1 188.8 mm to (176.6, 97.0)
- moved TP4 188.2 mm to (145.0, 120.4)
- moved C1 187.6 mm to (153.2, 105.2), turned to -90 degrees
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Routing:
- net /I2C1_SDA: track 0.00 -> 116.0 mm, vias 0 -> 3
- net /I2C1_SCL: track 0.00 -> 114.5 mm, vias 0 -> 3
- net VBUS: track 50.0 -> 118.7 mm, vias 4 -> 5
- net /D-: track 2.50 -> 69.0 mm, vias 0 -> 2
- net /D+: track 2.50 -> 68.9 mm, vias 0 -> 2
- net GND: track 53.1 -> 98.7 mm, vias 15 -> 20
- net SHELL_GND2: track 0.00 -> 28.2 mm
- net +3.3V: track 18.6 -> 45.9 mm, vias 4 -> 9
- net /NRST: track 0.00 -> 26.8 mm
- net /BOOT0 / SWCLK: track 14.8 -> 33.6 mm
- net /USART1_RX: track 0.00 -> 15.7 mm
- net /USART1_TX: track 0.00 -> 13.2 mm
- net /VREF+: track 0.00 -> 11.7 mm
- net Net-(U5-VDD): track 0.00 -> 5.72 mm
- net /RS_485/RS_485_A: track 46.9 -> 52.2 mm
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
Commit message: PCB V1 Terminee
Parts:
- removed R31, R33, R34, R35, R36, R37: 0, Resistor_SMD:R_0805_2012Metric
- added JP1: SolderJumper_3_Open, Jumper:SolderJumper-3_P1.3mm_Open_Pad1.0x1.5mm, F.Cu at (220.0, 91.8)
- added JP2: SolderJumper_3_Open, Jumper:SolderJumper-3_P1.3mm_Open_Pad1.0x1.5mm, F.Cu at (217.0, 91.8)
- added JP3: SolderJumper_3_Open, Jumper:SolderJumper-3_P1.3mm_Open_Pad1.0x1.5mm, F.Cu at (211.0, 91.8)
- added JP4: SolderJumper_3_Open, Jumper:SolderJumper-3_P1.3mm_Open_Pad1.0x1.5mm, F.Cu at (214.0, 91.8)
- R30, R32: value 0 -> 1k
- moved R30 61.5 mm to (200.0, 93.7), turned to 180 degrees
- moved R2 60.5 mm to (174.0, 102.4), turned to 90 degrees
- moved R32 58.5 mm to (200.0, 95.8), turned to 180 degrees
- moved R3 57.4 mm to (176.1, 102.4), turned to 90 degrees
- moved TP5 57.3 mm to (175.0, 112.0)
- moved TP7 56.1 mm to (175.0, 120.0)
- moved TP6 25.6 mm to (140.5, 86.0)
- moved TP16 8.06 mm to (199.0, 113.9)
- moved TP17 8.00 mm to (199.1, 122.0)
- moved J5 0.50 mm to (151.5, 88.0)
- moved J6 0.50 mm to (169.3, 121.0)
Connections:
- R30 pad 1: /RS_485/RJ_LED1_PIN1 -> Net-(JP1-A)
- R30 pad 2: +3.3V -> /USART1_RX
- R32 pad 1: /RS_485/RJ_LED2_PIN2 -> Net-(JP3-A)
- R32 pad 2: +3.3V -> /USART1_TX
Routing:
- net /USART1_TX: track 13.2 -> 154.4 mm
- net /USART1_RX: track 15.7 -> 147.2 mm, vias 0 -> 2
- net /CC1_ADC: track 1.88 -> 71.4 mm, vias 0 -> 2
- net /CC2_ADC: track 1.88 -> 71.2 mm, vias 0 -> 2
- net /PD0: track 0.00 -> 65.9 mm, vias 0 -> 3
- net /PD1: track 0.00 -> 64.8 mm, vias 0 -> 3
- net /PD2: track 0.00 -> 64.4 mm, vias 0 -> 3
- net /PD3: track 0.00 -> 63.8 mm, vias 0 -> 3
- net /USART1_DE: track 0.00 -> 60.8 mm, vias 0 -> 1
- net /PC13: track 0.00 -> 56.8 mm, vias 0 -> 4
- net Net-(J6-Pin_7): track 0.00 -> 50.8 mm, vias 0 -> 4
- net Net-(J6-Pin_8): track 0.00 -> 50.2 mm, vias 0 -> 4
- net /PF0: track 0.00 -> 48.0 mm, vias 0 -> 4
- net /SPI1_SCK: track 0.00 -> 44.5 mm
- net /SWDIO: track 0.00 -> 43.1 mm, vias 0 -> 3
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